Commit message: 修复仿真运动方向/转向 bug，新增网页定速巡航开关
- model.sdf/URDF：车轮关节轴向取反（原正指令实际后退），
  轮摩擦改各向异性(mu2=0.1+fdir1)修复滑移转向被摩擦锁死无法转向
- avoidance_node：enable_cruise/cruise_speed 支持运行时动态设置；
  期望方向可通行时直接采用，消除扇区量化导致的巡航持续右偏
- web_gateway/index.html：新增 POST /api/ugv/cruise 一键开关定速巡航，
  /api/status 上报避障状态，遥控页加巡航按钮
- README 同步网页巡航开关用法

File: CAR/CAR_ws/src/car_description/urdf/CAR_description.urdf (robot description, URDF)
Before this commit: robot r680_4wd, 9 links, 8 joints
Joints:
- joint front_left_wheel_joint: axis 0 -1 0 -> 0 1 0
- joint front_right_wheel_joint: axis 0 -1 0 -> 0 1 0
- joint rear_left_wheel_joint: axis 0 -1 0 -> 0 1 0
- joint rear_right_wheel_joint: axis 0 -1 0 -> 0 1 0

Commit message: CAR 适配阿克曼转向底盘（卖家发错货为阿克曼版 R680）
- 运动学改自行车模型：δ=atan2(ωL/v)，后轮速 v∓ω·track/2，v≈0 保护
- car_interfaces：新增 AckermannCommand（后轮双速+转向角），替换 WheelSpeeds
- chassis_controller/sim_motor_bridge/motor_driver 同步换算与话题 /ackermann_cmd
- avoidance_node：消除两处原地自旋指令，改带速弧线掉头（turn_speed）
- Gazebo 模型：前轮加转向节，diff-drive 插件换 ackermann-steering，URDF 同步
- 网页遥控：单指令互斥改组合按键，W+A 可同时控制驱动与转向（弧线行驶）
- 文档更新：README/HARDWARE_RESERVED（舵机零点备份、轴距/转向角待实测校准）

File: CAR/CAR_ws/src/car_description/urdf/CAR_description.urdf (robot description, URDF)
Before this commit: robot r680_4wd, 9 links, 8 joints
Links:
- added link front_left_steer_link, mass 0.3; visual box size=0.030 0.030 0.060
- added link front_right_steer_link, mass 0.3; visual box size=0.030 0.030 0.060
Joints:
- added joint front_left_steer_joint: type revolute, parent base_link, child front_left_steer_link, origin xyz=0.155 0.160 0 rpy=0 0 0, axis 0 0 1, limit lower=-0.5 upper=0.5 effort=5.0 velocity=5.0
- added joint front_right_steer_joint: type revolute, parent base_link, child front_right_steer_link, origin xyz=0.155 -0.160 0 rpy=0 0 0, axis 0 0 1, limit lower=-0.5 upper=0.5 effort=5.0 velocity=5.0
- joint front_left_wheel_joint: origin xyz=0.155 0.160 0 rpy=0 0 0 -> xyz=0 0 0 rpy=0 0 0; parent base_link -> front_left_steer_link
- joint front_right_wheel_joint: origin xyz=0.155 -0.160 0 rpy=0 0 0 -> xyz=0 0 0 rpy=0 0 0; parent base_link -> front_right_steer_link

Commit message: CAR v3.0：后置双摄像头、巡航转向辅助、N10P 激光雷达适配、一键仿真脚本
- 仿真/URDF 增加后置摄像头，web 遥控页前后双画面
- mux 新增 steering_assist：定速巡航中可手动转向
- 适配镭神 N10P 串口雷达（厂商 SDK vendored + 项目 launch/config）
- 新增 CAR/scripts/sim.sh 及 Windows 一键启停封装

File: CAR/CAR_ws/src/car_description/urdf/CAR_description.urdf (robot description, URDF)
Before this commit: robot r680_4wd, 11 links, 10 joints
Links:
- added link rear_camera_link, mass 0.080; collision box size=0.040 0.032 0.026; visual box size=0.040 0.032 0.026
- added link rear_camera_optical_frame, mass 0.001
Joints:
- added joint rear_camera_joint: type fixed, parent base_link, child rear_camera_link, origin xyz=-0.185 0 0.105 rpy=0 0 3.14159265359
- added joint rear_camera_optical_joint: type fixed, parent rear_camera_link, child rear_camera_optical_frame, origin xyz=0 0 0 rpy=-1.57079632679 0 -1.57079632679

Commit message: CAR：增加400mm停机坪并适配组合外廓避障

File: CAR/CAR_ws/src/car_description/urdf/CAR_description.urdf (robot description, URDF)
Before this commit: robot r680_4wd, 13 links, 12 joints
Links:
- added link landing_pad_link, mass 1.20; collision box size=0.400 0.400 0.012; visual box size=0.030 0.130 0.001
Joints:
- added joint landing_pad_joint: type fixed, parent base_link, child landing_pad_link, origin xyz=0 0 0.230 rpy=0 0 0

Commit message: CAR：停机坪居中机构全链路（ESP8266丝杆下位机 + Gazebo仿真 + 网页控制台）
- car_interfaces 新增 LeadscrewCommand/LeadscrewStatus 消息
- leadscrew_driver_node：双 T8 双向丝杆驱动（2×42步进，57mm 单边行程，
  状态机 AT_OUTER/AT_INNER/HOLD_MID + MOVING_IN/OUT），串口文本协议
  接 ESP8266 固件（tools/leadscrew42），simulate 模式同步驱动 Gazebo
  推杆关节；协议编解码独立为 esp_leadscrew_protocol.py
- Gazebo 模型：停机坪 400→450mm；A/B 边中点下方挂双出轴 42 步进 +
  T8 双向丝杆（末端±170mm）；4 个螺母+[型推杆一体 link（A/C 组 h1=30mm
  跨 A↔C，B/D 组 h2=55mm 跨 B↔D），4 个棱柱关节 + JointPositionController；
  螺母初始位于丝杆尽头（±160mm）；新增停机坪俯视相机
- 网页控制台：遥控页新增推杆开合键（POST /api/leadscrew/toggle，
  状态经 /api/status 轮询）；新增仿真专用监控台 /sim（标注仅用于仿真，
  俯视实时画面 + 推杆位置读数）
- 避障适配 450 坪：vehicle_half_width 0.20→0.225（节点默认值、两处
  launch、Nav2 备用 footprint 同步）
- WSL Humble 端到端验证：colcon 构建、指令→bridge→Gazebo 关节运动、
  网页按键全链路均实测通过

File: CAR/CAR_ws/src/car_description/urdf/CAR_description.urdf (robot description, URDF)
Before this commit: robot r680_4wd, 14 links, 13 joints
Links:
- link landing_pad_link: geometry collision box size=0.450 0.450 0.012; visual box size=0.030 0.130 0.001

Commit message: CAR：停机坪 470x470 + 居中机构几何更新（行程 57→67mm，电机加长至 60mm）
- 停机坪 450→470mm（SDF/URDF/模型描述/避障外廓半宽 0.235）
- 双出轴电机加长 40→60mm，丝杆自端面各伸 150mm 不变
  （含电机总长 360mm，末端 ±180mm）
- 螺母套外侧终点 ±170mm（齐平丝杆末端）、内侧 ±103mm，
  单边行程 57→67mm（53600 步/全程）：固件 TRAVEL_MM、节点默认参数、
  棱柱关节限位 [-0.067,0]、接口消息与网页读数联动
- 推杆横臂加长 460→480mm，垂腿外移至 ±240mm（坪边外侧 5mm）
- headless 仿真实测：避障 0.235、初始位 ±0.170、IN 全程
  精确到位 67.0mm/AT_INNER；固件 pio 编译通过

File: CAR/CAR_ws/src/car_description/urdf/CAR_description.urdf (robot description, URDF)
Before this commit: robot r680_4wd, 14 links, 13 joints
Links:
- link landing_pad_link: geometry collision box size=0.470 0.470 0.012; visual box size=0.030 0.130 0.001
